Commit message: adding ptu to rhodon URDF (include)

File: launch/rhodon/rhodon.xacro (robot description, xacro)
@@ -123,9 +123,16 @@
     <parent link="$(arg frame_ns)_base_link"/>
     <child link="$(arg frame_ns)_laser_front_link"/>
-    #
-    <origin_old rpy="3.14159 0 0" xyz="0.04 0.0 0.18"/>
-      # for SICK
-    <origin rpy="0 0 0" xyz="0.235 0.0 0.0"/>
-       # for hokuyo_urg
+    <!--<origin_old rpy="3.14159 0 0" xyz="0.04 0.0 0.18"/> --> # for SICK
+    <origin rpy="0 0 0" xyz="0.235 0.0 0.0"/>                   # for hokuyo_urg
+  </joint>
+  # PTU D46
+  <!-- Include and invoke the macro which creates a D46-->
+  <xacro:include filename="$(find hal_flir_d46)/urdf/d46.xacro" />
+  <xacro:ptu_d46 name="ptu" />
+  <!-- Create a fixed joint to connect the PTU to the rest of the robot -->
+  <joint name="base_to_ptu_base" type="fixed">
+    <parent link="$(arg frame_ns)_base_link"/>
+    <child link="ptu_base_link"/>
+    <origin xyz="0.15 0 0.8" rpy="0 0 0"/>
   </joint>
 </robot>

Commit message: adding interbotix ptu to rhodon xacro model

File: launch/rhodon/rhodon.xacro (robot description, xacro)
@@ -127,8 +127,8 @@
   </joint>
   # PTU D46
-  <!-- Include and invoke the macro which creates a D46-->
+  <!--
   <xacro:include filename="$(find hal_flir_d46)/urdf/d46.xacro" />
   <xacro:ptu_d46 name="ptu" />
-  <!-- Create a fixed joint to connect the PTU to the rest of the robot -->
+  # Create a fixed joint to connect the PTU to the rest of the robot
   <joint name="base_to_ptu_base" type="fixed">
     <parent link="$(arg frame_ns)_base_link"/>
@@ -136,3 +136,19 @@
     <origin xyz="0.15 0 0.8" rpy="0 0 0"/>
   </joint>
+  -->
+  # PTU WXXMS Interbotix
+  <xacro:include filename="$(find interbotix_xsturret_descriptions)/urdf/wxxms.urdf.xacro" />
+  # Create a fixed joint to connect the PTU to the rest of the robot
+  <joint name="base_to_ptu_base" type="fixed">
+    <parent link="$(arg frame_ns)_base_link"/>
+    <child link="wxxms/base_link"/>
+    <origin xyz="0.15 0 0.8" rpy="0 0 0"/>
+  </joint>
+  # Create a fixed joint to connect the Camera to the PTU
+  <link name="camera"/>
+  <joint name="camera_to_ptu_surface" type="fixed">
+    <parent link="wxxms/surface_link"/>
+    <child link="camera"/>
+    <origin xyz="0.0 0 0.0" rpy="-1.57079 0 -1.57079"/>
+  </joint>
 </robot>

Commit message: parking config

File: launch/rhodon/rhodon.xacro (robot description, xacro)
@@ -143,5 +143,5 @@
     <parent link="$(arg frame_ns)_base_link"/>
     <child link="wxxms/base_link"/>
-    <origin xyz="0.15 0 0.8" rpy="0 0 0"/>
+    <origin xyz="0.09 0.15 0.6" rpy="0 0 1.57079"/>
   </joint>
   # Create a fixed joint to connect the Camera to the PTU
@@ -150,5 +150,5 @@
     <parent link="wxxms/surface_link"/>
     <child link="camera"/>
-    <origin xyz="0.0 0 0.0" rpy="-1.57079 0 -1.57079"/>
+    <origin xyz="0.07 0 0.0" rpy="-1.57079 0 -1.57079"/>
   </joint>
 </robot>
