Commit message: updating methane launch

File: launch/methane/tdlas.xacro (robot description, xacro)
@@ -52,5 +52,5 @@
     <child link="camera"/>
     <!-- <origin xyz="0.07 0 0.0" rpy="-1.57079 0 -1.57079"/> -->
-    <origin xyz="0.07 0 0.0" rpy="-1.57079 -1.57079 -1.57079"/>
+    <origin xyz="0.0 0.095 0.11" rpy="-1.57079 -1.57079 -1.57079"/>
   </joint>
 </robot>

Commit message: PID controller and calibration (manual)

File: launch/methane/tdlas.xacro (robot description, xacro)
@@ -52,5 +52,5 @@
     <child link="camera"/>
     <!-- <origin xyz="0.07 0 0.0" rpy="-1.57079 0 -1.57079"/> -->
-    <origin xyz="0.0 0.095 0.11" rpy="-1.57079 -1.57079 -1.57079"/>
+    <origin xyz="0.0 0.092 0.05" rpy="-1.57079 -1.57079 -1.57079"/>
   </joint>
 </robot>

Commit message: new fix transform to set the TDLAS with respect a GPS

File: launch/methane/tdlas.xacro (robot description, xacro)
@@ -40,6 +40,13 @@
   # PTU WXXMS Interbotix
   <xacro:include filename="$(find interbotix_xsturret_descriptions)/urdf/wxxms.urdf.xacro" />
+  # Create a fixed joint to connect the BASE to the GPS
+  <link name="gps_tdlas"/>
+  <joint name="gps_to_base_joint" type="fixed">
+    <parent link="gps_tdlas"/>
+    <child link="$(arg frame_ns)_base_link"/>
+    <origin xyz="0.0 0.0 0.0" rpy="0 0 0"/>
+  </joint>
   # Create a fixed joint to connect the PTU to the base
-  <joint name="base_to_ptu_base" type="fixed">
+  <joint name="base_to_ptu_joint" type="fixed">
     <parent link="$(arg frame_ns)_base_link"/>
     <child link="wxxms/base_link"/>
